Commit message: feat: add arm_ik launch configuration and update yolo tracking and debug nodes

File: wildbot_workspace-main/workspaces/kros_car_persistent.xacro (robot description, xacro)
@@ -699,3 +699,17 @@
     <origin xyz="0.1 0 0.15" rpy="0 0 0"/>
   </joint>
+  <link name="camera_link">
+    <visual>
+      <origin xyz="0 0 0" rpy="0 0 0"/>
+      <geometry>
+        <box size="0.02 0.1 0.02"/>
+      </geometry>
+      <material name="silver"/>
+    </visual>
+  </link>
+  <joint name="camera_joint" type="fixed">
+    <parent link="base_link"/>
+    <child link="camera_link"/>
+    <origin xyz="0.15 0 0.3587" rpy="0 0 0"/>
+  </joint>
 </robot>

Commit message: Enhance YOLO 3D detection and arm IK integration
- Updated `ik_solver.py` to prioritize the use of a generated URDF file and added error handling for loading the robot description.
- Commented out debug logging in `debug_node.py` to reduce console output during operation.
- Implemented hardware height compensation in `detect_3d_node.py` to correct Z-axis discrepancies and adjusted depth filtering thresholds.
- Modified logging in `yolo_node.py` to provide more informative detection results while reducing unnecessary output.
- Added a new script `yolo_3d.sh` to streamline the launch of YOLO 3D detection mode with necessary configurations.
- Updated documentation to reflect the new 3D detection mode and its integration with the robotic arm's grab task functionality.
- Created a new markdown file detailing the IK and sensor compensation techniques used in the Wildbot system.

File: wildbot_workspace-main/workspaces/kros_car_persistent.xacro (robot description, xacro)
@@ -1,5 +1,5 @@
 <?xml version="1.0" ?>
 <robot name="kros_car" xmlns:xacro="http://www.ros.org/wiki/xacro">
-<xacro:include filename="materials.xacro" />
+<!-- <xacro:include filename="materials.xacro" /> -->
 <xacro:arg name="wheel_port" default="/dev/usb_wheel" />
 <xacro:arg name="wheel_baudrate" default="115200" />
@@ -510,17 +510,4 @@
 </joint>
 <joint name="Rigid 2" type="fixed">
-  <origin xyz="0.135 -0.127581 -0.000674" rpy="0 0 0"/>
-  <parent link="upper_blue_v1_1"/>
-  <child link="upper_silver_v1_1"/>
-</joint>
-<joint name="Rigid 3" type="fixed">
-  <origin xyz="-0.150487 0.0 0.074934" rpy="0 0 0"/>
-  <parent link="base_link"/>
-  <child link="Side_U_Bracket_Component1_v2_1"/>
-</joint>
-<joint name="Rigid 16" type="fixed">
-  <origin xyz="-0.007313 0.02025 -0.017533" rpy="0 0 0"/>
-  <parent link="Side_U_Bracket_Component1_v2_1"/>
-  <child link="new_motor_v2_1"/>
 </joint>
 <joint name="Rigid 27" type="fixed">
@@ -711,5 +698,5 @@
     <parent link="base_link"/>
     <child link="camera_link"/>
-    <origin xyz="0.15 0 0.3587" rpy="0 0 0"/>
+    <origin xyz="0.135 0 0.265" rpy="0 -0.523 0"/>
   </joint>
 </robot>

Commit message: Update robot workspace configuration

File: wildbot_workspace-main/workspaces/kros_car_persistent.xacro (robot description, xacro)
@@ -510,4 +510,17 @@
 </joint>
 <joint name="Rigid 2" type="fixed">
+  <origin xyz="0.134497 -0.127581 0.110239" rpy="0 0 0"/>
+  <parent link="base_link"/>
+  <child link="upper_silver_v1_1"/>
+</joint>
+<joint name="Rigid 3" type="fixed">
+  <origin xyz="-0.150487 0.0 0.074934" rpy="0 0 0"/>
+  <parent link="base_link"/>
+  <child link="Side_U_Bracket_Component1_v2_1"/>
+</joint>
+<joint name="Rigid 4" type="fixed">
+  <origin xyz="-0.007313 0.02025 -0.017533" rpy="0 0 0"/>
+  <parent link="Side_U_Bracket_Component1_v2_1"/>
+  <child link="new_motor_v2_1"/>
 </joint>
 <joint name="Rigid 27" type="fixed">
