Commit message: feat: add nav2 navigation stack and update arm poses and URDF joints

File: wildbot_workspace-main/kros_car.urdf (robot description, URDF)
Before this commit: robot kros_car, 26 links, 23 joints
Joints:
- added joint Rigid 3: type fixed, parent base_link, child Side_U_Bracket_Component1_v2_1, origin xyz=-0.150487 0.0 0.074934 rpy=0 0 0
- added joint Rigid 4: type fixed, parent Side_U_Bracket_Component1_v2_1, child new_motor_v2_1, origin xyz=-0.007313 0.02025 -0.017533 rpy=0 0 0
- joint Rigid 2: child (none) -> upper_silver_v1_1; origin (none) -> xyz=0.134497 -0.127581 0.110239 rpy=0 0 0; parent (none) -> base_link

Commit message: refactor: update tf2 library components and integrate new Foxglove bridge configuration scripts

File: wildbot_workspace-main/kros_car.urdf (robot description, URDF)
Before this commit: robot kros_car, 26 links, 25 joints
Links:
- added link base_footprint
- added link imu_link
Joints:
- added joint base_footprint_to_base_link: type fixed, parent base_footprint, child base_link, origin xyz=0 0 0.05 rpy=0 0 0
- added joint imu_joint: type fixed, parent base_link, child imu_link, origin xyz=0 0 0 rpy=0 0 0
- joint Rigid 3: origin xyz=-0.150487 0.0 0.074934 rpy=0 0 0 -> xyz=0.150487 0.0 0.074934 rpy=0 0 0
- joint laser_joint: origin xyz=0.1 0 0.15 rpy=0 0 0 -> xyz=-0.12 0 0.15 rpy=0 0 3.141592653589793

File: wildbot_workspace-main/workspaces/kros_car_persistent.xacro (robot description, xacro)
@@ -24,4 +24,10 @@
 <xacro:arg name="wheel_joints" default="wheel_1_joint,wheel_2_joint,wheel_3_joint,wheel_4_joint" />
 <xacro:arg name="arm_joints" default="arm_1_joint,arm_2_joint,gripper_joint" />
+<link name="base_footprint"/>
+<joint name="base_footprint_to_base_link" type="fixed">
+  <parent link="base_footprint"/>
+  <child link="base_link"/>
+  <origin xyz="0 0 0.05" rpy="0 0 0"/>
+</joint>
 <link name="base_link">
   <inertial>
@@ -515,5 +521,5 @@
 </joint>
 <joint name="Rigid 3" type="fixed">
-  <origin xyz="-0.150487 0.0 0.074934" rpy="0 0 0"/>
+  <origin xyz="0.150487 0.0 0.074934" rpy="0 0 0"/>
   <parent link="base_link"/>
   <child link="Side_U_Bracket_Component1_v2_1"/>
@@ -697,5 +703,11 @@
     <parent link="base_link"/>
     <child link="laser"/>
-    <origin xyz="0.1 0 0.15" rpy="0 0 0"/>
+    <origin xyz="-0.12 0 0.15" rpy="0 0 3.141592653589793"/>
+  </joint>
+  <link name="imu_link"/>
+  <joint name="imu_joint" type="fixed">
+    <parent link="base_link"/>
+    <child link="imu_link"/>
+    <origin xyz="0 0 0" rpy="0 0 0"/>
   </joint>
   <link name="camera_link">

Commit message: chore: update ros2_controllers repository dependencies, workflows, documentation, and test configurations

File: wildbot_workspace-main/kros_car.urdf (robot description, URDF)
Before this commit: robot kros_car, 28 links, 27 joints
Joints:
- joint arm_1_joint: axis 0.0 -1.0 0.0 -> 0.0 1.0 0.0; limit (none) -> effort=10.0 velocity=6.28; origin xyz=-0.007312 -0.01975 0.027605 rpy=3.14159265 1.04719755 -3.14159265 -> xyz=-0.007312 -0.01975 0.027605 rpy=3.14159265 1.04719755 0.0
- joint arm_2_joint: limit (none) -> effort=10.0 velocity=6.28
- joint camera_joint: origin xyz=0.135 0 0.265 rpy=0 -0.523 0 -> xyz=0.115862 0 0.186 rpy=0 0.523 0
- joint gripper_joint: limit (none) -> effort=10.0 velocity=6.28
- joint gripper_joint_2: limit (none) -> effort=10.0 velocity=6.28

File: wildbot_workspace-main/workspaces/kros_car_persistent.xacro (robot description, xacro)
@@ -2,4 +2,7 @@
 <robot name="kros_car" xmlns:xacro="http://www.ros.org/wiki/xacro">
 <!-- <xacro:include filename="materials.xacro" /> -->
+<material name="silver">
+  <color rgba="0.7 0.7 0.7 1.0"/>
+</material>
 <xacro:arg name="wheel_port" default="/dev/usb_wheel" />
 <xacro:arg name="wheel_baudrate" default="115200" />
@@ -595,8 +598,9 @@
 </joint>
 <joint name="arm_1_joint" type="continuous">
-  <origin xyz="-0.007312 -0.01975 0.027605" rpy="3.14159265 1.04719755 -3.14159265"/>
+  <origin xyz="-0.007312 -0.01975 0.027605" rpy="3.14159265 1.04719755 0.0"/>
   <parent link="new_motor_v2_1"/>
   <child link="big_U_self_v2_1"/>
-  <axis xyz="0.0 -1.0 0.0"/>
+  <axis xyz="0.0 1.0 0.0"/>
+  <limit effort="10.0" velocity="6.28"/>
 </joint>
 <joint name="Rigid 42" type="fixed">
@@ -615,4 +619,5 @@
   <child link="big_U_self_v2__1__1"/>
   <axis xyz="0.0 -1.0 -0.0"/>
+  <limit effort="10.0" velocity="6.28"/>
 </joint>
 <joint name="Rigid 45" type="fixed">
@@ -626,4 +631,5 @@
   <child link="grap2_v2_1"/>
   <axis xyz="-1.0 -0.0 -0.00037"/>
+  <limit effort="10.0" velocity="6.28"/>
 </joint>
 <joint name="gripper_joint_2" type="continuous">
@@ -632,4 +638,5 @@
   <child link="grap2_v2_Mirror__1"/>
   <axis xyz="1.0 0.0 0.00037"/>
+  <limit effort="10.0" velocity="6.28"/>
 </joint>
   <ros2_control name="kros_car_system" type="system">
@@ -723,5 +730,5 @@
     <parent link="base_link"/>
     <child link="camera_link"/>
-    <origin xyz="0.135 0 0.265" rpy="0 -0.523 0"/>
+    <origin xyz="0.115862 0 0.186" rpy="0 0.523 0"/>
   </joint>
 </robot>

Commit message: feat: add arm IK utilities, navigation debugging tools, and camera configuration updates

File: wildbot_workspace-main/kros_car.urdf (robot description, URDF)
Before this commit: robot kros_car, 28 links, 27 joints
Joints:
- joint camera_joint: origin xyz=0.115862 0 0.186 rpy=0 0.523 0 -> xyz=0.115862 0 0.278 rpy=0 0.262 0

File: wildbot_workspace-main/workspaces/kros_car_persistent.xacro (robot description, xacro)
@@ -730,5 +730,5 @@
     <parent link="base_link"/>
     <child link="camera_link"/>
-    <origin xyz="0.115862 0 0.186" rpy="0 0.523 0"/>
+    <origin xyz="0.115862 0 0.278" rpy="0 0.262 0"/>
   </joint>
 </robot>

Commit message: feat: add navigation and grabbing automation scripts, update map origin, and provide shorthand shell aliases for robot control

File: wildbot_workspace-main/kros_car.urdf (robot description, URDF)
Before this commit: robot kros_car, 28 links, 27 joints
Joints:
- joint camera_joint: origin xyz=0.115862 0 0.278 rpy=0 0.262 0 -> xyz=0.115862 0 0.29 rpy=0 0.384 0
- joint laser_joint: origin xyz=-0.12 0 0.15 rpy=0 0 3.141592653589793 -> xyz=-0.12 0 0.15 rpy=0 0 3.4906585

File: wildbot_workspace-main/workspaces/kros_car_persistent.xacro (robot description, xacro)
@@ -710,5 +710,5 @@
     <parent link="base_link"/>
     <child link="laser"/>
-    <origin xyz="-0.12 0 0.15" rpy="0 0 3.141592653589793"/>
+    <origin xyz="-0.12 0 0.15" rpy="0 0 3.4906585"/>
   </joint>
   <link name="imu_link"/>
@@ -730,5 +730,5 @@
     <parent link="base_link"/>
     <child link="camera_link"/>
-    <origin xyz="0.115862 0 0.278" rpy="0 0.262 0"/>
+    <origin xyz="0.115862 0 0.29" rpy="0 0.384 0"/>
   </joint>
 </robot>
